File: Itsy Bitsy 32u4 3V.brd (EAGLE design)
At the start: 35.6 x 17.8 mm, 26 parts, among them IC1 ATMEGA32U4-MU, IC2 74HCT1G125DBV, SW1 SPST_TACT-KMR2, U2 MIC5225-3.3, X3 microUSB, Y1 8MHz

Commit message: update 3V regulator label
Parts:
- U2: value MIC5225-3.3 -> AP2112K
Changed lines of the file:
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@@
 <?xml version="1.0" encoding="utf-8"?>
 <!DOCTYPE eagle SYSTEM "eagle.dtd">
-<eagle version="6.4">
+<eagle version="9.6.2">
 <drawing>
 <settings>
-<setting alwaysvectorfont="yes"/>
+<setting alwaysvectorfont="no"/>
+<setting keepoldvectorfont="yes"/>
 <setting verticaltext="up"/>
 </settings>
@@
 <layer number="59" name="tCarbon" color="7" fill="1" visible="no" active="no"/>
 <layer number="60" name="bCarbon" color="7" fill="1" visible="no" active="no"/>
-<layer number="90" name="Modules" color="7" fill="1" visible="no" active="yes"/>
+<layer number="90" name="Modules" color="7" fill="1" visible="no" active="no"/>
 <layer number="91" name="Nets" color="2" fill="1" visible="no" active="no"/>
 <layer number="92" name="Busses" color="1" fill="1" visible="no" active="no"/>
@@
 <param name="dpMaxLengthDifference" value="10mm"/>
 <param name="dpGapFactor" value="2.5"/>
-<param name="checkGrid" value="0"/>
 <param name="checkAngle" value="1"/>
 <param name="checkFont" value="1"/>
 <param name="checkRestrict" value="1"/>
+<param name="checkStop" value="0"/>
+<param name="checkValues" value="0"/>
+<param name="checkNames" value="1"/>
+<param name="checkWireStubs" value="1"/>
+<param name="checkPolygonWidth" value="0"/>
 <param name="useDiameter" value="13"/>
 <param name="maxErrors" value="50"/>
@@
 <pass name="Default">
 <param name="RoutingGrid" value="50mil"/>
+<param name="AutoGrid" value="1"/>
+<param name="Efforts" value="0"/>
+<param name="TopRouterVariant" value="1"/>
 <param name="tpViaShape" value="round"/>
 <param name="PrefDir.1" value="|"/>
@@
 <attribute name="COMPANY" value="ADAFRUIT INDUSTRIES" x="7.112" y="5.588" size="1.778" layer="27" rot="R90" display="off"/>
 <attribute name="DRAWN" value="KTOWN" x="7.112" y="5.588" size="1.778" layer="27" rot="R90" display="off"/>
+<attribute name="NAME" x="6.4245" y="7.458" size="0.8128" layer="25" ratio="18"/>
 <attribute name="REV" value="A" x="7.112" y="5.588" size="1.778" layer="27" rot="R90" display="off"/>
-<attribute name="NAME" x="6.4245" y="7.458" size="0.8128" layer="25" ratio="18"/>
 <attribute name="VALUE" x="7.49" y="4.2926" size="0.8128" layer="27" ratio="10" rot="R90"/>
 </element>
@@
 <attribute name="VALUE" x="0.448" y="11.541" size="0.8128" layer="27" ratio="10" rot="R270"/>
 </element>
-<element name="U2" library="microbuilder" package="SOT23-5" value="MIC5225-3.3" x="11.938" y="7.5692" smashed="yes" rot="R180">
+<element name="U2" library="microbuilder" package="SOT23-5" value="AP2112K" x="11.938" y="7.5692" smashed="yes" rot="R180">
 <attribute name="NAME" x="9.96" y="7.5692" size="0.8128" layer="25" ratio="18" rot="R180"/>
 <attribute name="VALUE" x="17.072" y="7.9502" size="0.8128" layer="27" ratio="10" rot="R180"/>
@@
 <contactref element="X3" pad="SPRT@4"/>
 <contactref element="X3" pad="BASE@1"/>
-<contactref element="X3" pad="SPRT@2"/>
-<contactref element="X3" pad="SPRT@1"/>
-<contactref element="X3" pad="GND"/>
-<contactref element="X3" pad="SPRT@3"/>
-<contactref element="X3" pad="BASE@2"/>
-<contactref element="X3" pad="SPRT@4"/>
-<contactref element="X3" pad="BASE@1"/>
 <contactref element="U2" pad="2"/>
 <contactref element="L" pad="C"/>
 <contactref element="JP2" pad="2"/>
-<contactref element="JP2" pad="2"/>
 <contactref element="IC2" pad="3"/>
 <contactref element="IC2" pad="1"/>
-<contactref element="IC2" pad="3"/>
 <wire x1="18.388015625" y1="5.2725875" x2="19.431" y2="6.315571875" width="0.2032" layer="1"/>
 <wire x1="19.431" y1="6.315571875" x2="19.431" y2="8.436890625" width="0.2032" layer="1"/>
@@
 <contactref element="IC1" pad="7"/>
 <contactref element="X3" pad="VBUS"/>
-<contactref element="X3" pad="VBUS"/>
 <contactref element="JP2" pad="3"/>
 <contactref element="D1" pad="A"/>
@@
 </signal>
 </signals>
+<mfgpreviewcolors>
+<mfgpreviewcolor name="soldermaskcolor" color="0xC8008000"/>
+<mfgpreviewcolor name="silkscreencolor" color="0xFFFEFEFE"/>
+<mfgpreviewcolor name="backgroundcolor" color="0xFF282828"/>
+<mfgpreviewcolor name="coppercolor" color="0xFFFFBF00"/>
+<mfgpreviewcolor name="substratecolor" color="0xFF786E46"/>
+</mfgpreviewcolors>
 </board>
 </drawing>
